File: Schematic_diagrams/BT_blockshelf/BT_blockshelf.kicad_sch (KiCad schematic)
At the start: 49 parts, among them SW1 SW_SPDT_MSM, SW2 SW_SPDT_MSM, SW3 SW_SPDT_MSM, SW4 SW_SPDT_MSM, SW5 SW_SPDT_MSM, SW6 SW_SPDT_MSM, SW7 SW_Push

Commit message: updates to rev B
Parts:
- added D3: SA12CA, symbol Device:D_TVS_Small_Filled
- D1, D2: value 1N4007 -> UF4007
Connections:
- net at 14.1, 1411.1, 1411.1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: now also D3.1 (A1)
- net at 13.1, 1412.1, D1.1 (K)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: now also D3.2 (A2)
Other:
- moved on the sheet: 13, 14, D1
