File: Schematic_diagrams/Common/Billingshurst2sheet2.kicad_sch (KiCad schematic)
At the start: 28 parts, among them U10 VCC, U11 GND, U12 EL817, U13 VCC, U14 GND, U15 VCC, U3 EL817, U4 GND, U5 VCC, U7 EL817, U8 GND, U9 EL817

Commit message: updates to rev B
Other:
- company: Amberley Museum - Billingshurst Signal Box -> Amerley Museum - Billingshurst Signalbox
- title: 4-Channel EL817 Optocoupler -> Track Diagram Lamp Controller
Changed lines of the file:
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@@
 	(paper "A4")
 	(title_block
-		(title "4-Channel EL817 Optocoupler")
-		(date "2026-02-09")
-		(rev "A")
-		(company "Amberley Museum - Billingshurst Signal Box")
+		(title "Track Diagram Lamp Controller")
+		(date "07/02/2026")
+		(rev "B")
+		(company "Amerley Museum - Billingshurst Signalbox")
 	)
 	(text_box "Channel 4 of 4-channel\noptocoupler module pcb\nAl-Zard DST-1R4P-N"

Commit message: Amberley spelling corrected
Other:
- company: Amerley Museum - Billingshurst Signalbox -> Amberley Museum - Billingshurst Signalbox
Changed lines of the file:
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@@
 		(date "07/02/2026")
 		(rev "B")
-		(company "Amerley Museum - Billingshurst Signalbox")
+		(company "Amberley Museum - Billingshurst Signalbox")
 	)
 	(text_box "Channel 4 of 4-channel\noptocoupler module pcb\nAl-Zard DST-1R4P-N"
