File: Schematic_diagrams/AHB_control_box/AHB_control_box.kicad_sch (KiCad schematic)
At the start: 3 parts, among them U1 4047

Commit message: cosmetic mods
cosmetic mods plus update to pdf
Parts:
- added A4: Quad_HG7881_H-Bridge_Module, symbol New_Library:Quad_HG7881_H-Bridge_Module
- added C6, C7: 4.7uF, symbol Device:C
- added R13, R14: 820k, symbol Device:R_Small
- added R15, R16, R17: 470R, symbol Device:R_Small
- added U2, U6: 4047 Monostable Multivibrator, symbol 4xxx:4047
- U1: value 4047 -> 4047 Monostable Multivibrator
Connections:
- net +5V: now also A4. (Motor_D), U2.14 (VDD), U2.4 (~{ASTABLE}), U6.14 (VDD), U6.4 (~{ASTABLE})
- net GND: now also A4. (Motor_D), U2.5 (ASTABLE), U2.6 (-TRIGGER), U2.7 (VSS), U2.9 (EXT_RESET), U6.5 (ASTABLE), U6.6 (-TRIGGER), U6.7 (VSS), U6.9 (EXT_RESET)
- net at U1.10 (Q): now also A4. (Motor_D)
- net at U1.11 (~{Q}): now also A4. (Motor_D)
- new net: C7.1, U6.1 (C)
- new net: C7.2, R14.2, U6.3 (RC_COMMON)
- new net: R14.1, U6.2 (R)
- new net: A4. (Motor_D), R16.1
- new net: A4. (Motor_D), U6.10 (Q)
- new net: A4. (Motor_D), U6.11 (~{Q})
- new net: A4. (Motor_D), R15.1
- new net: A4. (Motor_D), R17.1
- new net: A4. (Motor_D), U2.10 (Q)
- new net: A4. (Motor_D), U2.11 (~{Q})
- new net: R13.1, U2.2 (R)
- new net: C6.2, R13.2, U2.3 (RC_COMMON)
- new net: C6.1, U2.1 (C)
- new net Adversane: U2.12 (RETRIGGER), U2.8 (+TRIGGER)
- new net Adversane Repeater +: R16.2
- new net Adversane Repeater -: A4. (Motor_D)
- new net Barns Green: U6.12 (RETRIGGER), U6.8 (+TRIGGER)
- new net Barns Green Repeater +: R17.2
- new net Barns Green Repeater -: A4. (Motor_D)
- new net Cray Lane Repeater +: R15.2
- new net Cray Lane Repeater -: A4. (Motor_D)
Other:
- note added: "Quad_HG7881_H-Bridge_Module"
- title: (none) -> AHB Control Box
